File: KLON.kicad_pcb (KiCad board)
At the start: 2 copper layers, 68 parts, among them J1 Conn_01x03, J2 Conn_01x03, J3 Conn_01x02, SW1 3PDT, U1 TL072, U2 TL072

Commit message: updates. Going to temporarily remove ground connections in PCB file to make it easier to route.
Parts:
- added IC1: MAX1044ESA+, Housings_DIP:DIP-8_W7.62mm_Socket, F.Cu at (284.5, 106.7)
- moved D5 206.4 mm to (284.2, 94.0)
- moved Z1 201.7 mm to (296.0, 120.7), turned to 180 degrees
- moved D4 195.6 mm to (281.9, 85.1)
- moved C16 195.2 mm to (309.9, 94.0)
- moved C21 193.4 mm to (318.8, 94.0)
- moved C17 192.9 mm to (313.0, 102.9)
- moved C18 184.8 mm to (304.1, 102.9)
- moved D3 173.5 mm to (269.2, 108.0)
- moved C20 172.7 mm to (299.0, 94.0)
- moved C22 159.0 mm to (281.2, 101.6)
- moved C6 88.1 mm to (37.4, 41.9)
- moved U2 87.2 mm to (127.0, 95.2)
- moved C12 84.7 mm to (41.2, 63.5)
- moved R27 81.4 mm to (260.4, 97.8)
- moved C9 71.1 mm to (55.9, 44.5)
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
Commit message: Finished .kicad_pcb. Oshpark quote is $45 for 3 boards. Those cuts aren't pretty, but they are cheap.
Parts:
- moved C21 195.9 mm to (123.2, 106.4)
- moved R8 183.7 mm to (64.3, 105.9)
- moved R9 180.0 mm to (64.3, 102.4)
- moved C16 173.3 mm to (136.9, 105.2), turned to 270 degrees
- moved C20 168.4 mm to (130.9, 105.3), turned to 270 degrees
- moved C18 168.3 mm to (136.6, 86.2)
- moved R7 167.6 mm to (83.6, 106.5)
- moved C17 167.4 mm to (146.2, 88.2), turned to 180 degrees
- moved R5 166.0 mm to (62.7, 98.0)
- moved D3 163.1 mm to (107.1, 90.2), turned to 180 degrees
- moved R28 161.9 mm to (99.7, 132.0), turned to 180 degrees
- moved R17 160.0 mm to (76.4, 117.4)
- moved R25 159.7 mm to (76.4, 124.7)
- moved R29 159.2 mm to (89.5, 135.8)
- moved R26 157.1 mm to (76.5, 128.4)
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Routing:
- net V+: track 0.00 -> 167.2 mm, vias 0 -> 3
- net VB+: track 0.00 -> 153.8 mm, vias 0 -> 4
- net OUTPUT: track 0.00 -> 129.3 mm, vias 0 -> 1
- net POST-BUFF: track 0.00 -> 100.2 mm, vias 0 -> 1
- net S2-to-3PDT6: track 0.00 -> 71.5 mm
- net STAGE1-OUT: track 0.00 -> 71.1 mm, vias 0 -> 1
- net 3PDT-1: track 0.00 -> 64.3 mm, vias 0 -> 1
- net Net-(C19-Pad1): track 0.00 -> 63.9 mm
- net Net-(C8-Pad1): track 0.00 -> 62.0 mm
- net V2+: track 0.00 -> 56.5 mm, vias 0 -> 2
- net Net-(C7-Pad1): track 0.00 -> 45.7 mm, vias 0 -> 1
- net Net-(C3-Pad2): track 0.00 -> 42.9 mm
- net Net-(C13-Pad1): track 0.00 -> 41.6 mm
- net Net-(C11-Pad1): track 0.00 -> 38.2 mm
- net Net-(C14-Pad1): track 0.00 -> 36.4 mm, vias 0 -> 1
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- added copper zone on B.Cu, net GND
- added copper zone on F.Cu, net GND
Other:
- board outline added: 94.5 x 63.5 mm
- board text added: "3/25/2018"
- board text added: "enolk"
- board text added: "it ain't pretty, but oshpark made it cheap"
- board text added: "woof"
